Commit message: Add gpu flag to enable gpu simulation for launch file

File: urdf/livox_avia.xacro (robot description, xacro)
@@ -9,4 +9,5 @@
   <xacro:property name="samples" value="24000"/>
   <xacro:property name="downsample" value="1"/>
+  <xacro:arg name="gpu" default="true"/>
   <xacro:macro name="null_inertial">
     <inertial>
@@ -17,5 +18,6 @@
     </inertial>
   </xacro:macro>
-  <xacro:macro name="Livox_Mid_gazebo_sensor" params="visualize:=True update_rate:=10 resolution:=0.002 noise_mean:=0.0 noise_stddev:=0.01 name:=livox">
+  <!-- CPU Based simulation -->
+  <xacro:macro name="livox_mid_gazebo_sensor" params="visualize:=True update_rate:=10 resolution:=0.002 noise_mean:=0.0 noise_stddev:=0.01 name:=livox ros_topic:=scan">
     <gazebo reference="${name}">
       <sensor type="ray" name="laser_${name}">
@@ -60,5 +62,48 @@
     </gazebo>
   </xacro:macro>
-  <xacro:macro name="Livox_AVIA" params="visualize:=True name:=livox">
+  <!-- GPU Based simulation -->
+  <xacro:macro name="livox_mid_gpu_gazebo_sensor" params="visualize:=True update_rate:=10 resolution:=0.002 noise_mean:=0.0 noise_stddev:=0.01 name:=livox ros_topic:=scan">
+    <gazebo reference="${name}">
+      <sensor type="gpu_ray" name="laser_${name}">
+        <pose>0 0 0 0 0 0</pose>
+        <visualize>${visualize}</visualize>
+        <update_rate>${update_rate}</update_rate>
+        <sample_sensor>True</sample_sensor>
+        <sample_size>${samples}</sample_size>
+        <sample_csv_file>package://livox_laser_simulation/scan_mode/avia.csv</sample_csv_file>
+        <ray>
+          <scan>
+          <horizontal>
+          <samples>100</samples>
+          <resolution>1</resolution>
+          <min_angle>${-horizontal_fov/360*M_PI}</min_angle>
+          <max_angle>${horizontal_fov/360*M_PI}</max_angle>
+          </horizontal>
+          <vertical>
+          <samples>50</samples>
+          <resolution>1</resolution>
+          <min_angle>${-vertical_fov/360*M_PI}</min_angle>
+          <max_angle>${vertical_fov/360*M_PI}</max_angle>
+          </vertical>
+          </scan>
+          <range>
+          <min>${laser_min_range}</min>
+          <max>${laser_max_range}</max>
+          <resolution>${resolution}</resolution>
+          </range>
+          <noise>
+          <type>gaussian</type>
+          <mean>${noise_mean}</mean>
+          <stddev>${noise_stddev}</stddev>
+          </noise>
+        </ray>
+        <!-- This ray plgin is only for visualization. -->
+        <plugin name="gazebo_ros_gpu_laser_controller" filename="liblivox_laser_gpu_simulation.so">
+    		  <ros_topic>${ros_topic}</ros_topic>
+        </plugin>
+      </sensor>
+    </gazebo>
+  </xacro:macro>
+  <xacro:macro name="Livox_AVIA" params="visualize:=True name:=livox gpu_enabled:=$(arg gpu)">
     <link name="${name}_base">
       <xacro:null_inertial/>
@@ -86,5 +131,12 @@
       <origin rpy="0 0 0" xyz="0.0 0.0 0.0"/>
     </joint>
-    <xacro:Livox_Mid_gazebo_sensor name="${name}" visualize="${visualize}"/>
+    <xacro:if value="${gpu_enabled}">
+      <!-- GPU based simulation -->
+      <xacro:livox_mid_gpu_gazebo_sensor name="${name}" visualize="${visualize}" ros_topic="${ros_topic}"/>
+    </xacro:if>
+    <xacro:unless value="${gpu_enabled}">
+      <!-- CPU based simulation -->
+      <xacro:livox_mid_gazebo_sensor name="${name}" visualize="${visualize}" ros_topic="${ros_topic}"/>
+    </xacro:unless>
   </xacro:macro>
     <xacro:Livox_AVIA name="livox"/>

File: urdf/livox_horizon.xacro (robot description, xacro)
@@ -9,4 +9,5 @@
   <xacro:property name="samples" value="24000"/>
   <xacro:property name="downsample" value="1"/>
+  <xacro:arg name="gpu" default="true"/>
   <xacro:macro name="null_inertial">
     <inertial>
@@ -17,5 +18,6 @@
     </inertial>
   </xacro:macro>
-  <xacro:macro name="Livox_Mid_gazebo_sensor" params="visualize:=True update_rate:=10 resolution:=0.002 noise_mean:=0.0 noise_stddev:=0.01 name:=livox">
+  <!-- CPU Based simulation -->
+  <xacro:macro name="livox_mid_gazebo_sensor" params="visualize:=True update_rate:=10 resolution:=0.002 noise_mean:=0.0 noise_stddev:=0.01 name:=livox ros_topic:=scan">
     <gazebo reference="${name}">
       <sensor type="ray" name="laser_${name}">
@@ -60,5 +62,48 @@
     </gazebo>
   </xacro:macro>
-  <xacro:macro name="Livox_HORIZON" params="visualize:=True name:=livox">
+  <!-- GPU Based simulation -->
+  <xacro:macro name="livox_mid_gpu_gazebo_sensor" params="visualize:=True update_rate:=10 resolution:=0.002 noise_mean:=0.0 noise_stddev:=0.01 name:=livox ros_topic:=scan">
+    <gazebo reference="${name}">
+      <sensor type="gpu_ray" name="laser_${name}">
+        <pose>0 0 0 0 0 0</pose>
+        <visualize>${visualize}</visualize>
+        <update_rate>${update_rate}</update_rate>
+        <sample_sensor>True</sample_sensor>
+        <sample_size>${samples}</sample_size>
+        <sample_csv_file>package://livox_laser_simulation/scan_mode/horizon.csv</sample_csv_file>
+        <ray>
+          <scan>
+          <horizontal>
+          <samples>100</samples>
+          <resolution>1</resolution>
+          <min_angle>${-horizontal_fov/360*M_PI}</min_angle>
+          <max_angle>${horizontal_fov/360*M_PI}</max_angle>
+          </horizontal>
+          <vertical>
+          <samples>50</samples>
+          <resolution>1</resolution>
+          <min_angle>${-vertical_fov/360*M_PI}</min_angle>
+          <max_angle>${vertical_fov/360*M_PI}</max_angle>
+          </vertical>
+          </scan>
+          <range>
+          <min>${laser_min_range}</min>
+          <max>${laser_max_range}</max>
+          <resolution>${resolution}</resolution>
+          </range>
+          <noise>
+          <type>gaussian</type>
+          <mean>${noise_mean}</mean>
+          <stddev>${noise_stddev}</stddev>
+          </noise>
+        </ray>
+        <!-- This ray plgin is only for visualization. -->
+        <plugin name="gazebo_ros_gpu_laser_controller" filename="liblivox_laser_gpu_simulation.so">
+    		  <ros_topic>${ros_topic}</ros_topic>
+        </plugin>
+      </sensor>
+    </gazebo>
+  </xacro:macro>
+  <xacro:macro name="Livox_HORIZON" params="visualize:=False name:=livox gpu_enabled:=$(arg gpu)">
     <link name="${name}_base">
       <xacro:null_inertial/>
@@ -71,7 +116,9 @@
       </visual>
       <collision>
-		  <origin xyz="0 0 0" rpy="0 0 0" /> <geometry> <mesh
-		  filename="package://livox_laser_simulation/meshes/livox_mid40.dae">
-		  </mesh> </geometry>
+          <origin xyz="0 0 0" rpy="0 0 0" />
+          <geometry>
+          <mesh filename="package://livox_laser_simulation/meshes/livox_mid40.dae">
+          </mesh>
+          </geometry>
       </collision>
     </link>
@@ -84,5 +131,12 @@
       <origin rpy="0 0 0" xyz="0.0 0.0 0.0"/>
     </joint>
-    <xacro:Livox_Mid_gazebo_sensor name="${name}" visualize="${visualize}"/>
+    <xacro:if value="${gpu_enabled}">
+      <!-- GPU based simulation -->
+      <xacro:livox_mid_gpu_gazebo_sensor name="${name}" visualize="${visualize}" ros_topic="${ros_topic}"/>
+    </xacro:if>
+    <xacro:unless value="${gpu_enabled}">
+      <!-- CPU based simulation -->
+      <xacro:livox_mid_gazebo_sensor name="${name}" visualize="${visualize}" ros_topic="${ros_topic}"/>
+    </xacro:unless>
   </xacro:macro>
     <xacro:Livox_HORIZON name="livox"/>

File: urdf/livox_mid360.xacro (robot description, xacro)
@@ -5,10 +5,9 @@
   <xacro:property name="laser_max_range" value="200.0"/>
   <xacro:property name="horizontal_fov" value="360"/>
-  <xacro:property name="vertical_fov_min" value="-180.0"/>
-  <xacro:property name="vertical_fov_max" value="180.0"/>
+  <xacro:property name="vertical_fov" value="180.0"/>
   <xacro:property name="ros_topic" value="scan"/>
   <xacro:property name="samples" value="20000"/>
   <xacro:property name="downsample" value="1"/>
-  <xacro:property name="gpu_enabled" value="true"/>
+  <xacro:arg name="gpu" default="true"/>
   <xacro:macro name="null_inertial">
     <inertial>
@@ -19,51 +18,52 @@
     </inertial>
   </xacro:macro>
-  <!-- CPU Simulation -->
-  <xacro:macro name="livox_mid_gazebo_sensor" params="visualize:=False update_rate:=10 resolution:=0.002 noise_mean:=0.0 noise_stddev:=0.02 name:=livox ros_topic:=/scan">
+  <!-- CPU Based simulation -->
+  <xacro:macro name="livox_mid_gazebo_sensor" params="visualize:=False update_rate:=10 resolution:=0.002 noise_mean:=0.0 noise_stddev:=0.01 name:=livox ros_topic:=scan">
     <gazebo reference="${name}">
-      <sensor type="ray" name="${name}">
+      <sensor type="ray" name="laser_${name}">
         <pose>0 0 0 0 0 0</pose>
-        <visualize>false</visualize>
+        <visualize>${visualize}</visualize>
         <update_rate>${update_rate}</update_rate>
+        <!-- This ray plgin is only for visualization. -->
         <plugin name="gazebo_ros_laser_controller" filename="liblivox_laser_simulation.so">
-          <ray>
-            <scan>
-              <horizontal>
-                <samples>200</samples>
-                <resolution>1</resolution>
-                <min_angle>${-horizontal_fov/360*M_PI}</min_angle>
-                <max_angle>${horizontal_fov/360*M_PI}</max_angle>
-              </horizontal>
-              <vertical>
-                <samples>100</samples>
-                <resolution>1</resolution>
-                <min_angle>${vertical_fov_min/180*M_PI}</min_angle>
-                <max_angle>${vertical_fov_max/180*M_PI}</max_angle>
-              </vertical>
-            </scan>
-            <range>
-              <min>${laser_min_range}</min>
-              <max>${laser_max_range}</max>
-              <resolution>${resolution}</resolution>
-            </range>
-            <noise>
-              <type>gaussian</type>
-              <mean>${noise_mean}</mean>
-              <stddev>${noise_stddev}</stddev>
-            </noise>
-          </ray>
+			<ray>
+			  <scan>
+				<horizontal>
+				<samples>100</samples>
+				<resolution>1</resolution>
+				<min_angle>${-horizontal_fov/360*M_PI}</min_angle>
+				<max_angle>${horizontal_fov/360*M_PI}</max_angle>
+				</horizontal>
+				<vertical>
+				<samples>50</samples>
+				<resolution>1</resolution>
+				<min_angle>${-vertical_fov/360*M_PI}</min_angle>
+				<max_angle>${vertical_fov/360*M_PI}</max_angle>
+				</vertical>
+			  </scan>
+			  <range>
+				<min>${laser_min_range}</min>
+				<max>${laser_max_range}</max>
+				<resolution>${resolution}</resolution>
+			  </range>
+			  <noise>
+				<type>gaussian</type>
+				<mean>${noise_mean}</mean>
+				<stddev>${noise_stddev}</stddev>
+			  </noise>
+			</ray>
           <visualize>${visualize}</visualize>
-          <samples>${samples}</samples>
-          <downsample>${downsample}</downsample>
-          <csv_file_name>package://livox_laser_simulation/scan_mode/mid360.csv</csv_file_name>
-          <ros_topic>${ros_topic}</ros_topic>
+		  <samples>${samples}</samples>
+		  <downsample>${downsample}</downsample>
+		  <csv_file_name>package://livox_laser_simulation/scan_mode/mid360.csv</csv_file_name>
+		  <ros_topic>${ros_topic}</ros_topic>
         </plugin>
       </sensor>
     </gazebo>
   </xacro:macro>
-  <!-- GPU Simulation -->
-  <xacro:macro name="livox_mid_gazebo_gpu_sensor" params="visualize:=False update_rate:=10 samples:=20000 resolution:=0.002 noise_mean:=0.0 noise_stddev:=0.0 name:=livox ros_topic:=/scan">
+  <!-- GPU Based simulation -->
+  <xacro:macro name="livox_mid_gazebo_gpu_sensor" params="visualize:=False update_rate:=10 resolution:=0.002 noise_mean:=0.0 noise_stddev:=0.01 name:=livox ros_topic:=scan">
     <gazebo reference="${name}">
-      <sensor type="gpu_ray" name="${name}">
+      <sensor type="gpu_ray" name="laser_${name}">
         <pose>0 0 0 0 0 0</pose>
         <visualize>${visualize}</visualize>
@@ -74,16 +74,16 @@
         <ray>
           <scan>
-            <horizontal>
-              <samples>1</samples>
-              <resolution>1</resolution>
-              <min_angle>${-horizontal_fov/360*M_PI}</min_angle>
-              <max_angle>${horizontal_fov/360*M_PI}</max_angle>
-            </horizontal>
-            <vertical>
-              <samples>1</samples>
-              <resolution>1</resolution>
-              <min_angle>${vertical_fov_min/180*M_PI}</min_angle>
-              <max_angle>${vertical_fov_max/180*M_PI}</max_angle>
-            </vertical>
+          <horizontal>
+            <samples>1</samples>
+            <resolution>1</resolution>
+            <min_angle>${-horizontal_fov/360*M_PI}</min_angle>
+            <max_angle>${horizontal_fov/360*M_PI}</max_angle>
+          </horizontal>
+          <vertical>
+            <samples>1</samples>
+            <resolution>1</resolution>
+            <min_angle>${-vertical_fov/360*M_PI}</min_angle>
+            <max_angle>${vertical_fov/360*M_PI}</max_angle>
+          </vertical>
           </scan>
           <range>
@@ -99,33 +99,37 @@
         </ray>
         <!-- This ray plgin is only for visualization. -->
-        <plugin name="gazebo_ros_gpu_laser_controller" filename="liblivox_laser_gpu_simulation.so">
-          <ros_topic>${ros_topic}</ros_topic>
+        <plugin name="gazebo_ros_laser_controller" filename="liblivox_laser_gpu_simulation.so">
+		      <csv_file_name>package://livox_laser_simulation/scan_mode/mid360.csv</csv_file_name>
+		      <ros_topic>${ros_topic}</ros_topic>
         </plugin>
       </sensor>
     </gazebo>
   </xacro:macro>
-  <xacro:macro name="livox_mid360" params="visualize:=False name:=livox parent:=livox_base ros_topic:=/scan gpu_enabled:=False">
-    <!-- base -->
-    <joint name="${name}_joint" type="fixed">
-      <origin rpy="0 0 0" xyz="0.0 0.0 0.0"/>
-      <parent link="${parent}"/>
-      <child link="${name}_base"/>
-    </joint>
+  <xacro:macro name="Livox_Mid360" params="visualize:=False name:=livox gpu_enabled:=$(arg gpu)">
     <link name="${name}_base">
       <xacro:null_inertial/>
       <visual>
-        <origin xyz="0 0 0" rpy="0 0 0"/>
+        <origin xyz="0.00 0 0.00" rpy="0 0 0"/>
         <geometry>
-          <mesh filename="package://common_description/meshes/livox/livox_mid360.stl">
+          <mesh filename="package://livox_laser_simulation/meshes/livox_mid360.stl">
           </mesh>
         </geometry>
       </visual>
+      <collision>
+          <origin xyz="0 0 0" rpy="0 0 0" />
+          <geometry>
+          <mesh filename="package://livox_laser_simulation/meshes/livox_mid360.stl">
+          </mesh>
+          </geometry>
+      </collision>
     </link>
-    <joint name="${name}_base_mount_joint" type="fixed">
-      <origin rpy="0 0 0" xyz="0.0 0.0 0.047"/>
+    <link name="${name}">
+      <xacro:null_inertial/>
+    </link>
+    <joint name="${name}_to_${name}_base_joint" type="fixed">
       <parent link="${name}_base"/>
       <child link="${name}"/>
+      <origin rpy="0 0 0" xyz="0.0 0.0 0.047"/>
     </joint>
-    <link name="${name}"/>
     <xacro:if value="${gpu_enabled}">
       <!-- GPU based simulation -->
@@ -134,6 +138,9 @@
     <xacro:unless value="${gpu_enabled}">
       <!-- CPU based simulation -->
-      <xacro:livox_mid_gazebo_sensor name="${name}" visualize="True" ros_topic="${ros_topic}"/>
+      <xacro:livox_mid_gazebo_sensor name="${name}" visualize="${visualize}" ros_topic="${ros_topic}"/>
     </xacro:unless>
   </xacro:macro>
+    <xacro:Livox_Mid360 name="livox"/>
+  <xacro:include filename="$(find livox_laser_simulation)/urdf/standardrobots_oasis300.xacro"/>
+  <xacro:link_oasis name="oasis"/>
 </robot>

File: urdf/livox_mid40.xacro (robot description, xacro)
@@ -9,4 +9,5 @@
   <xacro:property name="samples" value="24000"/>
   <xacro:property name="downsample" value="1"/>
+  <xacro:arg name="gpu" default="true"/>
   <xacro:macro name="null_inertial">
     <inertial>
@@ -17,5 +18,6 @@
     </inertial>
   </xacro:macro>
-  <xacro:macro name="Livox_Mid_gazebo_sensor" params="visualize:=True update_rate:=10 resolution:=0.002 noise_mean:=0.0 noise_stddev:=0.01 name:=livox">
+  <!-- CPU Based simulation -->
+  <xacro:macro name="livox_mid_gazebo_sensor" params="visualize:=True update_rate:=10 resolution:=0.002 noise_mean:=0.0 noise_stddev:=0.01 name:=livox ros_topic:=scan">
     <gazebo reference="${name}">
       <sensor type="ray" name="laser_${name}">
@@ -60,5 +62,48 @@
     </gazebo>
   </xacro:macro>
-  <xacro:macro name="Livox_Mid40" params="visualize:=True name:=livox">
+  <!-- GPU Based simulation -->
+  <xacro:macro name="livox_mid_gpu_gazebo_sensor" params="visualize:=True update_rate:=10 resolution:=0.002 noise_mean:=0.0 noise_stddev:=0.01 name:=livox ros_topic:=scan">
+    <gazebo reference="${name}">
+      <sensor type="gpu_ray" name="laser_${name}">
+        <pose>0 0 0 0 0 0</pose>
+        <visualize>${visualize}</visualize>
+        <update_rate>${update_rate}</update_rate>
+        <sample_sensor>True</sample_sensor>
+        <sample_size>${samples}</sample_size>
+        <sample_csv_file>package://livox_laser_simulation/scan_mode/mid40.csv</sample_csv_file>
+        <ray>
+          <scan>
+          <horizontal>
+          <samples>100</samples>
+          <resolution>1</resolution>
+          <min_angle>${-horizontal_fov/360*M_PI}</min_angle>
+          <max_angle>${horizontal_fov/360*M_PI}</max_angle>
+          </horizontal>
+          <vertical>
+          <samples>50</samples>
+          <resolution>1</resolution>
+          <min_angle>${-vertical_fov/360*M_PI}</min_angle>
+          <max_angle>${vertical_fov/360*M_PI}</max_angle>
+          </vertical>
+          </scan>
+          <range>
+          <min>${laser_min_range}</min>
+          <max>${laser_max_range}</max>
+          <resolution>${resolution}</resolution>
+          </range>
+          <noise>
+          <type>gaussian</type>
+          <mean>${noise_mean}</mean>
+          <stddev>${noise_stddev}</stddev>
+          </noise>
+        </ray>
+        <!-- This ray plgin is only for visualization. -->
+        <plugin name="gazebo_ros_gpu_laser_controller" filename="liblivox_laser_gpu_simulation.so">
+    		  <ros_topic>${ros_topic}</ros_topic>
+        </plugin>
+      </sensor>
+    </gazebo>
+  </xacro:macro>
+  <xacro:macro name="Livox_Mid40" params="visualize:=True name:=livox gpu_enabled:=$(arg gpu)">
     <link name="${name}_base">
       <xacro:null_inertial/>
@@ -71,7 +116,9 @@
       </visual>
       <collision>
-		  <origin xyz="0 0 0" rpy="0 0 0" /> <geometry> <mesh
-		  filename="package://livox_laser_simulation/meshes/livox_mid40.dae">
-		  </mesh> </geometry>
+          <origin xyz="0 0 0" rpy="0 0 0" />
+          <geometry>
+          <mesh filename="package://livox_laser_simulation/meshes/livox_mid40.dae">
+          </mesh>
+          </geometry>
       </collision>
     </link>
@@ -84,5 +131,12 @@
       <origin rpy="0 0 0" xyz="0.0 0.0 0.0"/>
     </joint>
-    <xacro:Livox_Mid_gazebo_sensor name="${name}" visualize="${visualize}"/>
+    <xacro:if value="${gpu_enabled}">
+      <!-- GPU based simulation -->
+      <xacro:livox_mid_gpu_gazebo_sensor name="${name}" visualize="${visualize}" ros_topic="${ros_topic}"/>
+    </xacro:if>
+    <xacro:unless value="${gpu_enabled}">
+      <!-- CPU based simulation -->
+      <xacro:livox_mid_gazebo_sensor name="${name}" visualize="${visualize}" ros_topic="${ros_topic}"/>
+    </xacro:unless>
   </xacro:macro>
     <xacro:Livox_Mid40 name="livox"/>

File: urdf/livox_mid70.xacro (robot description, xacro)
@@ -9,4 +9,5 @@
   <xacro:property name="samples" value="10000"/>
   <xacro:property name="downsample" value="1"/>
+  <xacro:arg name="gpu" default="true"/>
   <xacro:macro name="null_inertial">
     <inertial>
@@ -17,5 +18,6 @@
     </inertial>
   </xacro:macro>
-  <xacro:macro name="Livox_Mid_gazebo_sensor" params="visualize:=True update_rate:=10 resolution:=0.002 noise_mean:=0.0 noise_stddev:=0.01 name:=livox">
+  <!-- CPU Based simulation -->
+  <xacro:macro name="livox_mid_gazebo_sensor" params="visualize:=True update_rate:=10 resolution:=0.002 noise_mean:=0.0 noise_stddev:=0.01 name:=livox ros_topic:=scan">
     <gazebo reference="${name}">
       <sensor type="ray" name="laser_${name}">
@@ -60,5 +62,48 @@
     </gazebo>
   </xacro:macro>
-  <xacro:macro name="Livox_Mid70" params="visualize:=True name:=livox">
+  <!-- GPU Based simulation -->
+  <xacro:macro name="livox_mid_gpu_gazebo_sensor" params="visualize:=True update_rate:=10 resolution:=0.002 noise_mean:=0.0 noise_stddev:=0.01 name:=livox ros_topic:=scan">
+    <gazebo reference="${name}">
+      <sensor type="gpu_ray" name="laser_${name}">
+        <pose>0 0 0 0 0 0</pose>
+        <visualize>${visualize}</visualize>
+        <update_rate>${update_rate}</update_rate>
+        <sample_sensor>True</sample_sensor>
+        <sample_size>${samples}</sample_size>
+        <sample_csv_file>package://livox_laser_simulation/scan_mode/mid70.csv</sample_csv_file>
+        <ray>
+          <scan>
+          <horizontal>
+          <samples>100</samples>
+          <resolution>1</resolution>
+          <min_angle>${-horizontal_fov/360*M_PI}</min_angle>
+          <max_angle>${horizontal_fov/360*M_PI}</max_angle>
+          </horizontal>
+          <vertical>
+          <samples>50</samples>
+          <resolution>1</resolution>
+          <min_angle>${-vertical_fov/360*M_PI}</min_angle>
+          <max_angle>${vertical_fov/360*M_PI}</max_angle>
+          </vertical>
+          </scan>
+          <range>
+          <min>${laser_min_range}</min>
+          <max>${laser_max_range}</max>
+          <resolution>${resolution}</resolution>
+          </range>
+          <noise>
+          <type>gaussian</type>
+          <mean>${noise_mean}</mean>
+          <stddev>${noise_stddev}</stddev>
+          </noise>
+        </ray>
+        <!-- This ray plgin is only for visualization. -->
+        <plugin name="gazebo_ros_gpu_laser_controller" filename="liblivox_laser_gpu_simulation.so">
+    		  <ros_topic>${ros_topic}</ros_topic>
+        </plugin>
+      </sensor>
+    </gazebo>
+  </xacro:macro>
+  <xacro:macro name="Livox_Mid70" params="visualize:=True name:=livox gpu_enabled:=$(arg gpu)">
     <link name="${name}_base">
       <xacro:null_inertial/>
@@ -86,5 +131,12 @@
       <origin rpy="0 0 0" xyz="0.0 0.0 0.0"/>
     </joint>
-    <xacro:Livox_Mid_gazebo_sensor name="${name}" visualize="${visualize}"/>
+    <xacro:if value="${gpu_enabled}">
+      <!-- GPU based simulation -->
+      <xacro:livox_mid_gpu_gazebo_sensor name="${name}" visualize="${visualize}" ros_topic="${ros_topic}"/>
+    </xacro:if>
+    <xacro:unless value="${gpu_enabled}">
+      <!-- CPU based simulation -->
+      <xacro:livox_mid_gazebo_sensor name="${name}" visualize="${visualize}" ros_topic="${ros_topic}"/>
+    </xacro:unless>
   </xacro:macro>
     <xacro:Livox_Mid70 name="livox"/>
