Commit message: Add gpu flag to enable gpu simulation for launch file

File: urdf/livox_tele.xacro (robot description, xacro)
@@ -9,4 +9,5 @@
   <xacro:property name="samples" value="24000"/>
   <xacro:property name="downsample" value="1"/>
+  <xacro:arg name="gpu" default="true"/>
   <xacro:macro name="null_inertial">
     <inertial>
@@ -17,5 +18,6 @@
     </inertial>
   </xacro:macro>
-  <xacro:macro name="Livox_Mid_gazebo_sensor" params="visualize:=True update_rate:=10 resolution:=0.002 noise_mean:=0.0 noise_stddev:=0.01 name:=livox">
+  <!-- CPU Based simulation -->
+  <xacro:macro name="livox_mid_gazebo_sensor" params="visualize:=True update_rate:=10 resolution:=0.002 noise_mean:=0.0 noise_stddev:=0.01 name:=livox ros_topic:=scan">
     <gazebo reference="${name}">
       <sensor type="ray" name="laser_${name}">
@@ -60,5 +62,48 @@
     </gazebo>
   </xacro:macro>
-  <xacro:macro name="Livox_TELE" params="visualize:=True name:=livox">
+  <!-- GPU Based simulation -->
+  <xacro:macro name="livox_mid_gpu_gazebo_sensor" params="visualize:=True update_rate:=10 resolution:=0.002 noise_mean:=0.0 noise_stddev:=0.01 name:=livox ros_topic:=scan">
+    <gazebo reference="${name}">
+      <sensor type="gpu_ray" name="laser_${name}">
+        <pose>0 0 0 0 0 0</pose>
+        <visualize>${visualize}</visualize>
+        <update_rate>${update_rate}</update_rate>
+        <sample_sensor>True</sample_sensor>
+        <sample_size>${samples}</sample_size>
+        <sample_csv_file>package://livox_laser_simulation/scan_mode/tele.csv</sample_csv_file>
+        <ray>
+          <scan>
+          <horizontal>
+          <samples>100</samples>
+          <resolution>1</resolution>
+          <min_angle>${-horizontal_fov/360*M_PI}</min_angle>
+          <max_angle>${horizontal_fov/360*M_PI}</max_angle>
+          </horizontal>
+          <vertical>
+          <samples>50</samples>
+          <resolution>1</resolution>
+          <min_angle>${-vertical_fov/360*M_PI}</min_angle>
+          <max_angle>${vertical_fov/360*M_PI}</max_angle>
+          </vertical>
+          </scan>
+          <range>
+          <min>${laser_min_range}</min>
+          <max>${laser_max_range}</max>
+          <resolution>${resolution}</resolution>
+          </range>
+          <noise>
+          <type>gaussian</type>
+          <mean>${noise_mean}</mean>
+          <stddev>${noise_stddev}</stddev>
+          </noise>
+        </ray>
+        <!-- This ray plgin is only for visualization. -->
+        <plugin name="gazebo_ros_gpu_laser_controller" filename="liblivox_laser_gpu_simulation.so">
+    		  <ros_topic>${ros_topic}</ros_topic>
+        </plugin>
+      </sensor>
+    </gazebo>
+  </xacro:macro>
+  <xacro:macro name="Livox_TELE" params="visualize:=True name:=livox gpu_enabled:=$(arg gpu)">
     <link name="${name}_base">
       <xacro:null_inertial/>
@@ -86,5 +131,12 @@
       <origin rpy="0 0 0" xyz="0.0 0.0 0.0"/>
     </joint>
-    <xacro:Livox_Mid_gazebo_sensor name="${name}" visualize="${visualize}"/>
+    <xacro:if value="${gpu_enabled}">
+      <!-- GPU based simulation -->
+      <xacro:livox_mid_gpu_gazebo_sensor name="${name}" visualize="${visualize}" ros_topic="${ros_topic}"/>
+    </xacro:if>
+    <xacro:unless value="${gpu_enabled}">
+      <!-- CPU based simulation -->
+      <xacro:livox_mid_gazebo_sensor name="${name}" visualize="${visualize}" ros_topic="${ros_topic}"/>
+    </xacro:unless>
   </xacro:macro>
     <xacro:Livox_TELE name="livox"/>
