Commit message: Fix xacro intentions
- use iterations to populate PointCloud2
- add missing iostream include

File: urdf/livox_avia.xacro (robot description, xacro)
@@ -25,37 +25,36 @@
         <visualize>${visualize}</visualize>
         <update_rate>${update_rate}</update_rate>
-        <!-- This ray plgin is only for visualization. -->
         <plugin name="gazebo_ros_laser_controller" filename="liblivox_laser_simulation.so">
-			<ray>
-			  <scan>
-				<horizontal>
-				<samples>100</samples>
-				<resolution>1</resolution>
-				<min_angle>${-horizontal_fov/360*M_PI}</min_angle>
-				<max_angle>${horizontal_fov/360*M_PI}</max_angle>
-				</horizontal>
-				<vertical>
-				<samples>50</samples>
-				<resolution>1</resolution>
-				<min_angle>${-vertical_fov/360*M_PI}</min_angle>
-				<max_angle>${vertical_fov/360*M_PI}</max_angle>
-				</vertical>
-			  </scan>
-			  <range>
-				<min>${laser_min_range}</min>
-				<max>${laser_max_range}</max>
-				<resolution>${resolution}</resolution>
-			  </range>
-			  <noise>
-				<type>gaussian</type>
-				<mean>${noise_mean}</mean>
-				<stddev>${noise_stddev}</stddev>
-			  </noise>
-			</ray>
+          <ray>
+            <scan>
+              <horizontal>
+                <samples>100</samples>
+                <resolution>1</resolution>
+                <min_angle>${-horizontal_fov/360*M_PI}</min_angle>
+                <max_angle>${horizontal_fov/360*M_PI}</max_angle>
+              </horizontal>
+              <vertical>
+                <samples>50</samples>
+                <resolution>1</resolution>
+                <min_angle>${-vertical_fov/360*M_PI}</min_angle>
+                <max_angle>${vertical_fov/360*M_PI}</max_angle>
+              </vertical>
+            </scan>
+            <range>
+              <min>${laser_min_range}</min>
+              <max>${laser_max_range}</max>
+              <resolution>${resolution}</resolution>
+            </range>
+            <noise>
+              <type>gaussian</type>
+              <mean>${noise_mean}</mean>
+              <stddev>${noise_stddev}</stddev>
+            </noise>
+          </ray>
           <visualize>${visualize}</visualize>
-		  <samples>${samples}</samples>
-		  <downsample>${downsample}</downsample>
-		  <csv_file_name>package://livox_laser_simulation/scan_mode/avia.csv</csv_file_name>
-		  <ros_topic>${ros_topic}</ros_topic>
+          <samples>${samples}</samples>
+          <downsample>${downsample}</downsample>
+          <csv_file_name>package://livox_laser_simulation/scan_mode/avia.csv</csv_file_name>
+          <ros_topic>${ros_topic}</ros_topic>
         </plugin>
       </sensor>
@@ -74,21 +73,21 @@
         <ray>
           <scan>
-          <horizontal>
-          <samples>100</samples>
-          <resolution>1</resolution>
-          <min_angle>${-horizontal_fov/360*M_PI}</min_angle>
-          <max_angle>${horizontal_fov/360*M_PI}</max_angle>
-          </horizontal>
-          <vertical>
-          <samples>50</samples>
-          <resolution>1</resolution>
-          <min_angle>${-vertical_fov/360*M_PI}</min_angle>
-          <max_angle>${vertical_fov/360*M_PI}</max_angle>
-          </vertical>
+            <horizontal>
+              <samples>100</samples>
+              <resolution>1</resolution>
+              <min_angle>${-horizontal_fov/360*M_PI}</min_angle>
+              <max_angle>${horizontal_fov/360*M_PI}</max_angle>
+            </horizontal>
+            <vertical>
+              <samples>50</samples>
+              <resolution>1</resolution>
+              <min_angle>${-vertical_fov/360*M_PI}</min_angle>
+              <max_angle>${vertical_fov/360*M_PI}</max_angle>
+            </vertical>
           </scan>
           <range>
-          <min>${laser_min_range}</min>
-          <max>${laser_max_range}</max>
-          <resolution>${resolution}</resolution>
+            <min>${laser_min_range}</min>
+            <max>${laser_max_range}</max>
+            <resolution>${resolution}</resolution>
           </range>
           <noise>
@@ -98,7 +97,6 @@
           </noise>
         </ray>
-        <!-- This ray plgin is only for visualization. -->
         <plugin name="gazebo_ros_gpu_laser_controller" filename="liblivox_laser_gpu_simulation.so">
-    		  <ros_topic>${ros_topic}</ros_topic>
+          <ros_topic>${ros_topic}</ros_topic>
         </plugin>
       </sensor>
@@ -111,14 +109,12 @@
         <origin xyz="0.00 0 0.00" rpy="0 0 0"/>
         <geometry>
-          <mesh filename="package://livox_laser_simulation/meshes/livox_mid40.dae">
-          </mesh>
+          <mesh filename="package://livox_laser_simulation/meshes/livox_mid40.dae"/>
         </geometry>
       </visual>
       <collision>
-          <origin xyz="0 0 0" rpy="0 0 0" />
-          <geometry>
-          <mesh filename="package://livox_laser_simulation/meshes/livox_mid40.dae">
-          </mesh>
-          </geometry>
+        <origin xyz="0 0 0" rpy="0 0 0" />
+        <geometry>
+          <mesh filename="package://livox_laser_simulation/meshes/livox_mid40.dae"/>
+        </geometry>
       </collision>
     </link>
@@ -140,5 +136,5 @@
     </xacro:unless>
   </xacro:macro>
-    <xacro:Livox_AVIA name="livox"/>
+  <xacro:Livox_AVIA name="livox"/>
   <xacro:include filename="$(find livox_laser_simulation)/urdf/standardrobots_oasis300.xacro"/>
   <xacro:link_oasis name="oasis"/>

File: urdf/livox_horizon.xacro (robot description, xacro)
@@ -25,37 +25,36 @@
         <visualize>${visualize}</visualize>
         <update_rate>${update_rate}</update_rate>
-        <!-- This ray plgin is only for visualization. -->
         <plugin name="gazebo_ros_laser_controller" filename="liblivox_laser_simulation.so">
-			<ray>
-			  <scan>
-				<horizontal>
-				<samples>100</samples>
-				<resolution>1</resolution>
-				<min_angle>${-horizontal_fov/360*M_PI}</min_angle>
-				<max_angle>${horizontal_fov/360*M_PI}</max_angle>
-				</horizontal>
-				<vertical>
-				<samples>50</samples>
-				<resolution>1</resolution>
-				<min_angle>${-vertical_fov/360*M_PI}</min_angle>
-				<max_angle>${vertical_fov/360*M_PI}</max_angle>
-				</vertical>
-			  </scan>
-			  <range>
-				<min>${laser_min_range}</min>
-				<max>${laser_max_range}</max>
-				<resolution>${resolution}</resolution>
-			  </range>
-			  <noise>
-				<type>gaussian</type>
-				<mean>${noise_mean}</mean>
-				<stddev>${noise_stddev}</stddev>
-			  </noise>
-			</ray>
+          <ray>
+            <scan>
+              <horizontal>
+                <samples>100</samples>
+                <resolution>1</resolution>
+                <min_angle>${-horizontal_fov/360*M_PI}</min_angle>
+                <max_angle>${horizontal_fov/360*M_PI}</max_angle>
+              </horizontal>
+              <vertical>
+                <samples>50</samples>
+                <resolution>1</resolution>
+                <min_angle>${-vertical_fov/360*M_PI}</min_angle>
+                <max_angle>${vertical_fov/360*M_PI}</max_angle>
+              </vertical>
+            </scan>
+            <range>
+              <min>${laser_min_range}</min>
+              <max>${laser_max_range}</max>
+              <resolution>${resolution}</resolution>
+            </range>
+            <noise>
+              <type>gaussian</type>
+              <mean>${noise_mean}</mean>
+              <stddev>${noise_stddev}</stddev>
+            </noise>
+          </ray>
           <visualize>${visualize}</visualize>
-		  <samples>${samples}</samples>
-		  <downsample>${downsample}</downsample>
-		  <csv_file_name>package://livox_laser_simulation/scan_mode/horizon.csv</csv_file_name>
-		  <ros_topic>${ros_topic}</ros_topic>
+          <samples>${samples}</samples>
+          <downsample>${downsample}</downsample>
+          <csv_file_name>package://livox_laser_simulation/scan_mode/horizon.csv</csv_file_name>
+          <ros_topic>${ros_topic}</ros_topic>
         </plugin>
       </sensor>
@@ -74,31 +73,30 @@
         <ray>
           <scan>
-          <horizontal>
-          <samples>100</samples>
-          <resolution>1</resolution>
-          <min_angle>${-horizontal_fov/360*M_PI}</min_angle>
-          <max_angle>${horizontal_fov/360*M_PI}</max_angle>
-          </horizontal>
-          <vertical>
-          <samples>50</samples>
-          <resolution>1</resolution>
-          <min_angle>${-vertical_fov/360*M_PI}</min_angle>
-          <max_angle>${vertical_fov/360*M_PI}</max_angle>
-          </vertical>
+            <horizontal>
+              <samples>100</samples>
+              <resolution>1</resolution>
+              <min_angle>${-horizontal_fov/360*M_PI}</min_angle>
+              <max_angle>${horizontal_fov/360*M_PI}</max_angle>
+            </horizontal>
+            <vertical>
+              <samples>50</samples>
+              <resolution>1</resolution>
+              <min_angle>${-vertical_fov/360*M_PI}</min_angle>
+              <max_angle>${vertical_fov/360*M_PI}</max_angle>
+            </vertical>
           </scan>
           <range>
-          <min>${laser_min_range}</min>
-          <max>${laser_max_range}</max>
-          <resolution>${resolution}</resolution>
+            <min>${laser_min_range}</min>
+            <max>${laser_max_range}</max>
+            <resolution>${resolution}</resolution>
           </range>
           <noise>
-          <type>gaussian</type>
-          <mean>${noise_mean}</mean>
-          <stddev>${noise_stddev}</stddev>
+            <type>gaussian</type>
+            <mean>${noise_mean}</mean>
+            <stddev>${noise_stddev}</stddev>
           </noise>
         </ray>
-        <!-- This ray plgin is only for visualization. -->
         <plugin name="gazebo_ros_gpu_laser_controller" filename="liblivox_laser_gpu_simulation.so">
-    		  <ros_topic>${ros_topic}</ros_topic>
+          <ros_topic>${ros_topic}</ros_topic>
         </plugin>
       </sensor>
@@ -111,14 +109,12 @@
         <origin xyz="0.00 0 0.00" rpy="0 0 0"/>
         <geometry>
-          <mesh filename="package://livox_laser_simulation/meshes/livox_mid40.dae">
-          </mesh>
+          <mesh filename="package://livox_laser_simulation/meshes/livox_mid40.dae"/>
         </geometry>
       </visual>
       <collision>
-          <origin xyz="0 0 0" rpy="0 0 0" />
-          <geometry>
-          <mesh filename="package://livox_laser_simulation/meshes/livox_mid40.dae">
-          </mesh>
-          </geometry>
+        <origin xyz="0 0 0" rpy="0 0 0" />
+        <geometry>
+          <mesh filename="package://livox_laser_simulation/meshes/livox_mid40.dae"/>
+        </geometry>
       </collision>
     </link>
@@ -140,5 +136,5 @@
     </xacro:unless>
   </xacro:macro>
-    <xacro:Livox_HORIZON name="livox"/>
+  <xacro:Livox_HORIZON name="livox"/>
   <xacro:include filename="$(find livox_laser_simulation)/urdf/standardrobots_oasis300.xacro"/>
   <xacro:link_oasis name="oasis"/>

File: urdf/livox_mid360.xacro (robot description, xacro)
@@ -25,37 +25,36 @@
         <visualize>${visualize}</visualize>
         <update_rate>${update_rate}</update_rate>
-        <!-- This ray plgin is only for visualization. -->
         <plugin name="gazebo_ros_laser_controller" filename="liblivox_laser_simulation.so">
-			<ray>
-			  <scan>
-				<horizontal>
-				<samples>100</samples>
-				<resolution>1</resolution>
-				<min_angle>${-horizontal_fov/360*M_PI}</min_angle>
-				<max_angle>${horizontal_fov/360*M_PI}</max_angle>
-				</horizontal>
-				<vertical>
-				<samples>50</samples>
-				<resolution>1</resolution>
-				<min_angle>${-vertical_fov/360*M_PI}</min_angle>
-				<max_angle>${vertical_fov/360*M_PI}</max_angle>
-				</vertical>
-			  </scan>
-			  <range>
-				<min>${laser_min_range}</min>
-				<max>${laser_max_range}</max>
-				<resolution>${resolution}</resolution>
-			  </range>
-			  <noise>
-				<type>gaussian</type>
-				<mean>${noise_mean}</mean>
-				<stddev>${noise_stddev}</stddev>
-			  </noise>
-			</ray>
+          <ray>
+            <scan>
+              <horizontal>
+                <samples>100</samples>
+                <resolution>1</resolution>
+                <min_angle>${-horizontal_fov/360*M_PI}</min_angle>
+                <max_angle>${horizontal_fov/360*M_PI}</max_angle>
+              </horizontal>
+              <vertical>
+                <samples>50</samples>
+                <resolution>1</resolution>
+                <min_angle>${-vertical_fov/360*M_PI}</min_angle>
+                <max_angle>${vertical_fov/360*M_PI}</max_angle>
+              </vertical>
+            </scan>
+            <range>
+              <min>${laser_min_range}</min>
+              <max>${laser_max_range}</max>
+              <resolution>${resolution}</resolution>
+            </range>
+            <noise>
+              <type>gaussian</type>
+              <mean>${noise_mean}</mean>
+              <stddev>${noise_stddev}</stddev>
+            </noise>
+          </ray>
           <visualize>${visualize}</visualize>
-		  <samples>${samples}</samples>
-		  <downsample>${downsample}</downsample>
-		  <csv_file_name>package://livox_laser_simulation/scan_mode/mid360.csv</csv_file_name>
-		  <ros_topic>${ros_topic}</ros_topic>
+          <samples>${samples}</samples>
+          <downsample>${downsample}</downsample>
+          <csv_file_name>package://livox_laser_simulation/scan_mode/mid360.csv</csv_file_name>
+          <ros_topic>${ros_topic}</ros_topic>
         </plugin>
       </sensor>
@@ -74,16 +73,16 @@
         <ray>
           <scan>
-          <horizontal>
-            <samples>1</samples>
-            <resolution>1</resolution>
-            <min_angle>${-horizontal_fov/360*M_PI}</min_angle>
-            <max_angle>${horizontal_fov/360*M_PI}</max_angle>
-          </horizontal>
-          <vertical>
-            <samples>1</samples>
-            <resolution>1</resolution>
-            <min_angle>${-vertical_fov/360*M_PI}</min_angle>
-            <max_angle>${vertical_fov/360*M_PI}</max_angle>
-          </vertical>
+            <horizontal>
+              <samples>1</samples>
+              <resolution>1</resolution>
+              <min_angle>${-horizontal_fov/360*M_PI}</min_angle>
+              <max_angle>${horizontal_fov/360*M_PI}</max_angle>
+            </horizontal>
+            <vertical>
+              <samples>1</samples>
+              <resolution>1</resolution>
+              <min_angle>${-vertical_fov/360*M_PI}</min_angle>
+              <max_angle>${vertical_fov/360*M_PI}</max_angle>
+            </vertical>
           </scan>
           <range>
@@ -98,8 +97,6 @@
           </noise>
         </ray>
-        <!-- This ray plgin is only for visualization. -->
         <plugin name="gazebo_ros_laser_controller" filename="liblivox_laser_gpu_simulation.so">
-		      <csv_file_name>package://livox_laser_simulation/scan_mode/mid360.csv</csv_file_name>
-		      <ros_topic>${ros_topic}</ros_topic>
+          <ros_topic>${ros_topic}</ros_topic>
         </plugin>
       </sensor>
@@ -112,14 +109,12 @@
         <origin xyz="0.00 0 0.00" rpy="0 0 0"/>
         <geometry>
-          <mesh filename="package://livox_laser_simulation/meshes/livox_mid360.stl">
-          </mesh>
+          <mesh filename="package://livox_laser_simulation/meshes/livox_mid360.stl"/>
         </geometry>
       </visual>
       <collision>
-          <origin xyz="0 0 0" rpy="0 0 0" />
-          <geometry>
-          <mesh filename="package://livox_laser_simulation/meshes/livox_mid360.stl">
-          </mesh>
-          </geometry>
+        <origin xyz="0 0 0" rpy="0 0 0" />
+        <geometry>
+          <mesh filename="package://livox_laser_simulation/meshes/livox_mid360.stl"/>
+        </geometry>
       </collision>
     </link>

File: urdf/livox_mid40.xacro (robot description, xacro)
@@ -25,37 +25,36 @@
         <visualize>${visualize}</visualize>
         <update_rate>${update_rate}</update_rate>
-        <!-- This ray plgin is only for visualization. -->
         <plugin name="gazebo_ros_laser_controller" filename="liblivox_laser_simulation.so">
-			<ray>
-			  <scan>
-				<horizontal>
-				<samples>100</samples>
-				<resolution>1</resolution>
-				<min_angle>${-horizontal_fov/360*M_PI}</min_angle>
-				<max_angle>${horizontal_fov/360*M_PI}</max_angle>
-				</horizontal>
-				<vertical>
-				<samples>50</samples>
-				<resolution>1</resolution>
-				<min_angle>${-vertical_fov/360*M_PI}</min_angle>
-				<max_angle>${vertical_fov/360*M_PI}</max_angle>
-				</vertical>
-			  </scan>
-			  <range>
-				<min>${laser_min_range}</min>
-				<max>${laser_max_range}</max>
-				<resolution>${resolution}</resolution>
-			  </range>
-			  <noise>
-				<type>gaussian</type>
-				<mean>${noise_mean}</mean>
-				<stddev>${noise_stddev}</stddev>
-			  </noise>
-			</ray>
+          <ray>
+            <scan>
+              <horizontal>
+                <samples>100</samples>
+                <resolution>1</resolution>
+                <min_angle>${-horizontal_fov/360*M_PI}</min_angle>
+                <max_angle>${horizontal_fov/360*M_PI}</max_angle>
+              </horizontal>
+              <vertical>
+                <samples>50</samples>
+                <resolution>1</resolution>
+                <min_angle>${-vertical_fov/360*M_PI}</min_angle>
+                <max_angle>${vertical_fov/360*M_PI}</max_angle>
+              </vertical>
+            </scan>
+            <range>
+              <min>${laser_min_range}</min>
+              <max>${laser_max_range}</max>
+              <resolution>${resolution}</resolution>
+            </range>
+            <noise>
+              <type>gaussian</type>
+              <mean>${noise_mean}</mean>
+              <stddev>${noise_stddev}</stddev>
+            </noise>
+          </ray>
           <visualize>${visualize}</visualize>
-		  <samples>${samples}</samples>
-		  <downsample>${downsample}</downsample>
-		  <csv_file_name>package://livox_laser_simulation/scan_mode/mid40.csv</csv_file_name>
-		  <ros_topic>${ros_topic}</ros_topic>
+          <samples>${samples}</samples>
+          <downsample>${downsample}</downsample>
+          <csv_file_name>package://livox_laser_simulation/scan_mode/mid40.csv</csv_file_name>
+          <ros_topic>${ros_topic}</ros_topic>
         </plugin>
       </sensor>
@@ -74,31 +73,31 @@
         <ray>
           <scan>
-          <horizontal>
-          <samples>100</samples>
-          <resolution>1</resolution>
-          <min_angle>${-horizontal_fov/360*M_PI}</min_angle>
-          <max_angle>${horizontal_fov/360*M_PI}</max_angle>
-          </horizontal>
-          <vertical>
-          <samples>50</samples>
-          <resolution>1</resolution>
-          <min_angle>${-vertical_fov/360*M_PI}</min_angle>
-          <max_angle>${vertical_fov/360*M_PI}</max_angle>
-          </vertical>
+            <horizontal>
+              <samples>100</samples>
+              <resolution>1</resolution>
+              <min_angle>${-horizontal_fov/360*M_PI}</min_angle>
+              <max_angle>${horizontal_fov/360*M_PI}</max_angle>
+            </horizontal>
+            <vertical>
+              <samples>50</samples>
+              <resolution>1</resolution>
+              <min_angle>${-vertical_fov/360*M_PI}</min_angle>
+              <max_angle>${vertical_fov/360*M_PI}</max_angle>
+            </vertical>
           </scan>
           <range>
-          <min>${laser_min_range}</min>
-          <max>${laser_max_range}</max>
-          <resolution>${resolution}</resolution>
+            <min>${laser_min_range}</min>
+            <max>${laser_max_range}</max>
+            <resolution>${resolution}</resolution>
           </range>
           <noise>
-          <type>gaussian</type>
-          <mean>${noise_mean}</mean>
-          <stddev>${noise_stddev}</stddev>
+            <type>gaussian</type>
+            <mean>${noise_mean}</mean>
+            <stddev>${noise_stddev}</stddev>
           </noise>
         </ray>
         <!-- This ray plgin is only for visualization. -->
         <plugin name="gazebo_ros_gpu_laser_controller" filename="liblivox_laser_gpu_simulation.so">
-    		  <ros_topic>${ros_topic}</ros_topic>
+          <ros_topic>${ros_topic}</ros_topic>
         </plugin>
       </sensor>
@@ -111,14 +110,12 @@
         <origin xyz="0.00 0 0.00" rpy="0 0 0"/>
         <geometry>
-          <mesh filename="package://livox_laser_simulation/meshes/livox_mid40.dae">
-          </mesh>
+          <mesh filename="package://livox_laser_simulation/meshes/livox_mid40.dae"/>
         </geometry>
       </visual>
       <collision>
-          <origin xyz="0 0 0" rpy="0 0 0" />
-          <geometry>
-          <mesh filename="package://livox_laser_simulation/meshes/livox_mid40.dae">
-          </mesh>
-          </geometry>
+        <origin xyz="0 0 0" rpy="0 0 0" />
+        <geometry>
+          <mesh filename="package://livox_laser_simulation/meshes/livox_mid40.dae"/>
+        </geometry>
       </collision>
     </link>
@@ -140,5 +137,5 @@
     </xacro:unless>
   </xacro:macro>
-    <xacro:Livox_Mid40 name="livox"/>
+  <xacro:Livox_Mid40 name="livox"/>
   <xacro:include filename="$(find livox_laser_simulation)/urdf/standardrobots_oasis300.xacro"/>
   <xacro:link_oasis name="oasis"/>
