Commit message: Fix cpu based simulation and add gpu based into xacro file

File: urdf/livox_mid360.xacro (robot description, xacro)
@@ -4,55 +4,23 @@
   <xacro:property name="laser_min_range" value="0.1"/>
   <xacro:property name="laser_max_range" value="200.0"/>
-  <xacro:property name="horizontal_fov" value="70.4"/>
-  <xacro:property name="vertical_fov" value="70.4"/>
+  <xacro:property name="horizontal_fov" value="360"/>
+  <xacro:property name="vertical_fov_min" value="-180.0"/>
+  <xacro:property name="vertical_fov_max" value="180.0"/>
   <xacro:property name="ros_topic" value="scan"/>
-  <xacro:property name="samples" value="10000"/>
+  <xacro:property name="samples" value="20000"/>
   <xacro:property name="downsample" value="1"/>
-  <xacro:macro name="null_inertial">
-    <inertial>
-      <mass value="0.1"/>
-    <inertia ixx="0.01" ixy="0" ixz="0"
-          iyy="0.01" iyz="0"
-          izz="0.01"/>
-    </inertial>
-  </xacro:macro>
-  <xacro:macro name="Livox_Mid_gazebo_sensor" params="visualize:=True update_rate:=10 resolution:=0.002 noise_mean:=0.0 noise_stddev:=0.0 name:=livox">
+  <xacro:property name="gpu_enabled" value="true"/>
+  <!-- CPU Simulation -->
+  <xacro:macro name="livox_mid_gazebo_sensor" params="visualize:=False update_rate:=10 resolution:=0.002 noise_mean:=0.0 noise_stddev:=0.02 name:=livox ros_topic:=/scan">
     <gazebo reference="${name}">
-      <sensor type="ray" name="laser_${name}">
+      <sensor type="ray" name="${name}">
         <pose>0 0 0 0 0 0</pose>
-        <visualize>${visualize}</visualize>
+        <visualize>false</visualize>
         <update_rate>${update_rate}</update_rate>
-        <ray>
-          <scan>
-            <horizontal>
-              <samples>100</samples>
-              <resolution>1</resolution>
-              <min_angle>${-horizontal_fov/360*M_PI}</min_angle>
-              <max_angle>${horizontal_fov/360*M_PI}</max_angle>
-            </horizontal>
-            <vertical>
-              <samples>50</samples>
-              <resolution>1</resolution>
-              <min_angle>${-vertical_fov/360*M_PI}</min_angle>
-              <max_angle>${vertical_fov/360*M_PI}</max_angle>
-            </vertical>
-          </scan>
-          <range>
-            <min>${laser_min_range}</min>
-            <max>${laser_max_range}</max>
-            <resolution>${resolution}</resolution>
-          </range>
-          <noise>
-            <type>gaussian</type>
-            <mean>${noise_mean}</mean>
-            <stddev>${noise_stddev}</stddev>
-          </noise>
-        </ray>
-        <!-- This ray plgin is only for visualization. -->
         <plugin name="gazebo_ros_laser_controller" filename="liblivox_laser_simulation.so">
           <ray>
             <scan>
               <horizontal>
-                <samples>100</samples>
+                <samples>200</samples>
                 <resolution>1</resolution>
                 <min_angle>${-horizontal_fov/360*M_PI}</min_angle>
@@ -60,8 +28,8 @@
               </horizontal>
               <vertical>
-                <samples>50</samples>
+                <samples>100</samples>
                 <resolution>1</resolution>
-                <min_angle>${-vertical_fov/360*M_PI}</min_angle>
-                <max_angle>${vertical_fov/360*M_PI}</max_angle>
+                <min_angle>${vertical_fov_min/180*M_PI}</min_angle>
+                <max_angle>${vertical_fov_max/180*M_PI}</max_angle>
               </vertical>
             </scan>
@@ -86,34 +54,77 @@
     </gazebo>
   </xacro:macro>
-  <xacro:macro name="Livox_Mid360" params="visualize:=True name:=livox">
+  <!-- GPU Simulation -->
+  <xacro:macro name="livox_mid_gazebo_gpu_sensor" params="visualize:=False update_rate:=10 samples:=20000 resolution:=0.002 noise_mean:=0.0 noise_stddev:=0.0 name:=livox ros_topic:=/scan">
+    <gazebo reference="${name}">
+      <sensor type="gpu_ray" name="${name}">
+        <pose>0 0 0 0 0 0</pose>
+        <visualize>${visualize}</visualize>
+        <update_rate>${update_rate}</update_rate>
+        <sample_sensor>True</sample_sensor>
+        <sample_size>${samples}</sample_size>
+        <sample_csv_file>package://livox_laser_simulation/scan_mode/mid360.csv</sample_csv_file>
+        <ray>
+          <scan>
+            <horizontal>
+              <samples>1</samples>
+              <resolution>1</resolution>
+              <min_angle>${-horizontal_fov/360*M_PI}</min_angle>
+              <max_angle>${horizontal_fov/360*M_PI}</max_angle>
+            </horizontal>
+            <vertical>
+              <samples>1</samples>
+              <resolution>1</resolution>
+              <min_angle>${vertical_fov_min/180*M_PI}</min_angle>
+              <max_angle>${vertical_fov_max/180*M_PI}</max_angle>
+            </vertical>
+          </scan>
+          <range>
+            <min>${laser_min_range}</min>
+            <max>${laser_max_range}</max>
+            <resolution>${resolution}</resolution>
+          </range>
+          <noise>
+            <type>gaussian</type>
+            <mean>${noise_mean}</mean>
+            <stddev>${noise_stddev}</stddev>
+          </noise>
+        </ray>
+        <!-- This ray plgin is only for visualization. -->
+        <plugin name="gazebo_ros_gpu_laser_controller" filename="liblivox_laser_gpu_simulation.so">
+          <ros_topic>${ros_topic}</ros_topic>
+        </plugin>
+      </sensor>
+    </gazebo>
+  </xacro:macro>
+  <xacro:macro name="livox_mid360" params="visualize:=False name:=livox parent:=livox_base ros_topic:=/scan gpu_enabled:=False">
+    <!-- base -->
+    <joint name="${name}_joint" type="fixed">
+      <origin rpy="0 0 0" xyz="0.0 0.0 0.0"/>
+      <parent link="${parent}"/>
+      <child link="${name}_base"/>
+    </joint>
     <link name="${name}_base">
-      <xacro:null_inertial/>
       <visual>
-        <origin xyz="0.00 0 0.00" rpy="0 0 0"/>
+        <origin xyz="0 0 0" rpy="0 0 0"/>
         <geometry>
-          <mesh filename="package://livox_laser_simulation/meshes/livox_mid40.dae">
+          <mesh filename="package://common_description/meshes/livox/livox_mid360.stl">
           </mesh>
         </geometry>
       </visual>
-      <collision>
-          <origin xyz="0 0 0" rpy="0 0 0" />
-          <geometry>
-          <mesh filename="package://livox_laser_simulation/meshes/livox_mid40.dae">
-          </mesh>
-          </geometry>
-      </collision>
     </link>
-    <link name="${name}">
-      <xacro:null_inertial/>
-    </link>
-    <joint name="${name}_to_${name}_base_joint" type="fixed">
+    <joint name="${name}_base_mount_joint" type="fixed">
+      <origin rpy="0 0 0" xyz="0.0 0.0 0.047"/>
       <parent link="${name}_base"/>
       <child link="${name}"/>
-      <origin rpy="0 0 0" xyz="0.0 0.0 0.0"/>
     </joint>
-    <xacro:Livox_Mid_gazebo_sensor name="${name}" visualize="${visualize}"/>
+    <link name="${name}"/>
+    <xacro:if value="${gpu_enabled}">
+      <!-- GPU based simulation -->
+      <xacro:livox_mid_gazebo_gpu_sensor name="${name}" visualize="${visualize}" ros_topic="${ros_topic}"/>
+    </xacro:if>
+    <xacro:unless value="${gpu_enabled}">
+      <!-- CPU based simulation -->
+      <xacro:livox_mid_gazebo_sensor name="${name}" visualize="True" ros_topic="${ros_topic}"/>
+    </xacro:unless>
   </xacro:macro>
-    <xacro:Livox_Mid360 name="livox"/>
-  <xacro:include filename="$(find livox_laser_simulation)/urdf/standardrobots_oasis300.xacro"/>
-  <xacro:link_oasis name="oasis"/>
 </robot>

Commit message: Remove unneccessary SendRosTf function

File: urdf/livox_mid360.xacro (robot description, xacro)
@@ -11,4 +11,12 @@
   <xacro:property name="downsample" value="1"/>
   <xacro:property name="gpu_enabled" value="true"/>
+  <xacro:macro name="null_inertial">
+    <inertial>
+      <mass value="0.1"/>
+    <inertia ixx="0.01" ixy="0" ixz="0"
+          iyy="0.01" iyz="0"
+          izz="0.01"/>
+    </inertial>
+  </xacro:macro>
   <!-- CPU Simulation -->
   <xacro:macro name="livox_mid_gazebo_sensor" params="visualize:=False update_rate:=10 resolution:=0.002 noise_mean:=0.0 noise_stddev:=0.02 name:=livox ros_topic:=/scan">
@@ -105,4 +113,5 @@
     </joint>
     <link name="${name}_base">
+      <xacro:null_inertial/>
       <visual>
         <origin xyz="0 0 0" rpy="0 0 0"/>

Commit message: Add parameter for publishing non-return rays and marker

File: urdf/livox_mid360.xacro (robot description, xacro)
@@ -7,4 +7,5 @@
   <xacro:property name="vertical_fov" value="180.0"/>
   <xacro:property name="ros_topic" value="scan"/>
+  <xacro:property name="ros_non_return_topic" value="non_return_rays"/>
   <xacro:property name="samples" value="20000"/>
   <xacro:property name="downsample" value="1"/>
@@ -19,5 +20,5 @@
   </xacro:macro>
   <!-- CPU Based simulation -->
-  <xacro:macro name="livox_mid_gazebo_sensor" params="visualize:=False update_rate:=10 resolution:=0.002 noise_mean:=0.0 noise_stddev:=0.01 name:=livox ros_topic:=scan">
+  <xacro:macro name="livox_mid_gazebo_sensor" params="visualize:=False update_rate:=10 resolution:=0.002 noise_mean:=0.0 noise_stddev:=0.01 name:=livox ros_topic:=scan ros_non_return_topic:=non_return_rays">
     <gazebo reference="${name}">
       <sensor type="ray" name="laser_${name}">
@@ -57,4 +58,5 @@
           <csv_file_name>package://livox_laser_simulation/scan_mode/mid360.csv</csv_file_name>
           <ros_topic>${ros_topic}</ros_topic>
+          <ros_non_return_topic>${ros_non_return_topic}</ros_non_return_topic>
         </plugin>
       </sensor>
@@ -133,5 +135,5 @@
     <xacro:unless value="${gpu_enabled}">
       <!-- CPU based simulation -->
-      <xacro:livox_mid_gazebo_sensor name="${name}" visualize="${visualize}" ros_topic="${ros_topic}"/>
+      <xacro:livox_mid_gazebo_sensor name="${name}" visualize="${visualize}" ros_topic="${ros_topic}" ros_non_return_topic="${ros_non_return_topic}"/>
     </xacro:unless>
   </xacro:macro>
